Commit message: remove joint loop to tool0

File: staubli_tx2-90_support/urdf/tx2-90l_macro.xacro (robot description, xacro)
@@ -231,9 +231,4 @@
     <!-- ROS-Industrial 'tool0' frame: all-zeros tool frame -->
     <link name="${prefix}tool0" />
-    <joint name="${prefix}flange-tool0" type="fixed">
-      <origin xyz="0 0 0" rpy="0 ${radians(90.0)} 0" />
-      <parent link="${prefix}flange" />
-      <child link="${prefix}tool0" />
-    </joint>
   </xacro:macro>
 </robot>

Commit message: add other tx2-90 variants

File: staubli_tx2-90_support/urdf/tx2-90l_macro.xacro (robot description, xacro)
@@ -8,12 +8,12 @@
         <origin xyz="0 0 0" rpy="0 0 0"/>
         <geometry>
-          <mesh filename="package://staubli_tx2-90_support/meshes/tx2-90l/visual/base_link.stl"/>
-        </geometry>
-        <xacro:material_staubli_ral_melon_yellow />
-      </visual>
-      <collision>
-        <origin xyz="0 0 0" rpy="0 0 0"/>
-        <geometry>
-          <mesh filename="package://staubli_tx2-90_support/meshes/tx2-90l/collision/base_link.stl"/>
+          <mesh filename="package://staubli_tx2-90_support/meshes/tx2-90/visual/base_link.stl"/>
+        </geometry>
+        <xacro:material_staubli_ral_melon_yellow />
+      </visual>
+      <collision>
+        <origin xyz="0 0 0" rpy="0 0 0"/>
+        <geometry>
+          <mesh filename="package://staubli_tx2-90_support/meshes/tx2-90/collision/base_link.stl"/>
         </geometry>
       </collision>
@@ -30,12 +30,12 @@
         <origin xyz="0 0 0" rpy="0 0 0"/>
         <geometry>
-          <mesh filename="package://staubli_tx2-90_support/meshes/tx2-90l/visual/link_1.stl"/>
-        </geometry>
-        <xacro:material_staubli_ral_melon_yellow />
-      </visual>
-      <collision>
-        <origin xyz="0 0 0" rpy="0 0 0"/>
-        <geometry>
-          <mesh filename="package://staubli_tx2-90_support/meshes/tx2-90l/collision/link_1.stl"/>
+          <mesh filename="package://staubli_tx2-90_support/meshes/tx2-90/visual/link_1.stl"/>
+        </geometry>
+        <xacro:material_staubli_ral_melon_yellow />
+      </visual>
+      <collision>
+        <origin xyz="0 0 0" rpy="0 0 0"/>
+        <geometry>
+          <mesh filename="package://staubli_tx2-90_support/meshes/tx2-90/collision/link_1.stl"/>
         </geometry>
       </collision>
@@ -74,12 +74,12 @@
         <origin xyz="0 0 0" rpy="0 0 0"/>
         <geometry>
-          <mesh filename="package://staubli_tx2-90_support/meshes/tx2-90l/visual/link_3.stl"/>
-        </geometry>
-        <xacro:material_staubli_ral_melon_yellow />
-      </visual>
-      <collision>
-        <origin xyz="0 0 0" rpy="0 0 0"/>
-        <geometry>
-          <mesh filename="package://staubli_tx2-90_support/meshes/tx2-90l/collision/link_3.stl"/>
+          <mesh filename="package://staubli_tx2-90_support/meshes/tx2-90/visual/link_3.stl"/>
+        </geometry>
+        <xacro:material_staubli_ral_melon_yellow />
+      </visual>
+      <collision>
+        <origin xyz="0 0 0" rpy="0 0 0"/>
+        <geometry>
+          <mesh filename="package://staubli_tx2-90_support/meshes/tx2-90/collision/link_3.stl"/>
         </geometry>
       </collision>
@@ -118,5 +118,5 @@
         <origin xyz="0 0 0" rpy="0 0 0"/>
         <geometry>
-          <mesh filename="package://staubli_tx2-90_support/meshes/tx2-90l/visual/link_5.stl"/>
+          <mesh filename="package://staubli_tx2-90_support/meshes/tx2-90/visual/link_5.stl"/>
         </geometry>
         <xacro:material_staubli_ral_grey_aluminium />
@@ -125,5 +125,5 @@
         <origin xyz="0 0 0" rpy="0 0 0"/>
         <geometry>
-          <mesh filename="package://staubli_tx2-90_support/meshes/tx2-90l/collision/link_5.stl"/>
+          <mesh filename="package://staubli_tx2-90_support/meshes/tx2-90/collision/link_5.stl"/>
         </geometry>
       </collision>
@@ -140,5 +140,5 @@
         <origin xyz="0 0 0" rpy="0 0 0"/>
         <geometry>
-          <mesh filename="package://staubli_tx2-90_support/meshes/tx2-90l/visual/link_6.stl"/>
+          <mesh filename="package://staubli_tx2-90_support/meshes/tx2-90/visual/link_6.stl"/>
         </geometry>
         <xacro:material_staubli_ral_grey_aluminium />
@@ -147,5 +147,5 @@
         <origin xyz="0 0 0" rpy="0 0 0"/>
         <geometry>
-          <mesh filename="package://staubli_tx2-90_support/meshes/tx2-90l/collision/link_6.stl"/>
+          <mesh filename="package://staubli_tx2-90_support/meshes/tx2-90/collision/link_6.stl"/>
         </geometry>
       </collision>
